File: StreamerPad.kicad_pcb (KiCad board)
At the start: 2 copper layers, 66.7 x 82 mm, 20 parts, among them U1 MOUDLE-SEEEDUINO-XIAO, U2 ER_OLEDM0.91_1x-I2C

Commit message: DAY05 PCB and Schematic (ver. 2)
Parts:
- added G***: LOGO, FERN:fern2, B.Cu at (135.7, 54.8)
- moved U2 2.38 mm to (87.3, 58.6)
- moved U1 1.90 mm to (135.7, 54.5)
Routing:
- net Column 1: track 132.0 -> 109.7 mm
- net Column 2: track 145.8 -> 124.9 mm
- net VCC: track 90.3 -> 72.9 mm
- net Column 0: track 116.3 -> 100.3 mm
- net SCL: track 58.0 -> 43.3 mm
- net GND: track 64.8 -> 75.4 mm
- net SDA: track 51.7 -> 43.3 mm
- net Row 2: track 108.4 -> 106.8 mm
- net Row 1: track 86.4 -> 85.3 mm
- net Row 0: track 64.3 -> 63.4 mm
- added copper zone on B.Cu, net (none)
- added copper zone on F.Cu, net (none)
Other:
- board text added: "JENNIE <3"
